File: PCB/Wisp5_Harvester_Motor-driver/Wisp5_Harvester_Motor-driver.brd (EAGLE design)
At the start: 100 x 80 mm, 29 parts

Commit message: Redone previous work, with more focus on power routing.
Parts:
- removed R13: 1.82M, resistor:R0805
- removed R14: 5.9M, resistor:R0805
- removed R15: 5.49M, resistor:R0805
- removed U$2: BQ25570, texas:VQFN20
- added R10: 6.49M, resistor:R0805
- added R3, R4: 10K, resistor:R0805
- added U1: BQ25570, texas:VQFN20
- R1: value 10K -> 8.66M
- R2: value 10K -> 4.30M
- R6: value 8.66M -> 1.82M
- R7: value 4.30M -> 5.9M
- R8: value 6.49M -> 5.49M
- moved R1 25.6 mm to (12.2, 26.5), turned to 180 degrees
- moved R2 17.7 mm to (10.3, 22.8), turned to 0 degrees
- moved C6 8.77 mm to (18.4, 17.4), turned to 0 degrees
- moved C7 8.23 mm to (23.5, 17.4), turned to 180 degrees
- moved C8 7.29 mm to (13.7, 16.4), turned to 90 degrees
- moved L2 6.97 mm to (9.35, 18.9)
- moved R9 6.37 mm to (3.65, 21.0)
- moved VIN/GND 6.14 mm to (24.7, 26.9), turned to 180 degrees
- moved R7 6.12 mm to (3.69, 26.9)
- moved R8 6.09 mm to (3.69, 24.1)
- moved R6 5.53 mm to (7.34, 26.0), turned to 270 degrees
- moved C3 3.50 mm to (27.3, 20.8)
- moved L1 2.97 mm to (23.2, 22.2)
- moved C1 2.65 mm to (6.80, 14.9), turned to 180 degrees
- moved DRV2 1.80 mm to (20.3, 13.6)
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- renumbered U$1 to U2
Connections:
- net GND: now also R10.1, R2.1, U1.1, U1.15, U1.17, U1.5, U1.9, U1.PWR_PAD, U1.PWR_PAD1, U1.PWR_PAD2, U1.PWR_PAD3, U1.PWR_PAD4; no longer R15.1, R7.1, U$2.1, U$2.15, U$2.17, U$2.5, U$2.9, U$2.PWR_PAD, U$2.PWR_PAD1, U$2.PWR_PAD2, U$2.PWR_PAD3, U$2.PWR_PAD4
- net N$1: now also R10.2, U1.12; no longer R8.2, U$2.12
- net N$10: now also R6.1, R7.2, U1.10; no longer R13.1, R14.2, U$2.10
- net N$12: now also U1.16; no longer U$2.16
- net N$13: now also R1.1, R2.2, U1.7; no longer R6.1, R7.2, U$2.7
- net N$18: now also R7.1, R8.2, U1.11; no longer R14.1, R15.2, U$2.11
- net N$2: now also R1.2, U1.8; no longer R13.2, U$2.8
- net N$4: now also U1.20; no longer U$2.20
- net N$9: now also U1.4; no longer U$2.4
- net SCL: now also R4.1; no longer R2.1
- net SDA: now also R3.1; no longer R1.1
- net VBAT: now also U1.18; no longer U$2.18
- net VBAT_OK: now also U1.13, U1.6; no longer U$2.13, U$2.6
- net VBUCK: now also R3.2, R4.2, U1.14; no longer R1.2, R2.2, U$2.14
- net VHARV: now also U1.2; no longer U$2.2
- net VSTOR: now also U1.19, U1.3; no longer U$2.19, U$2.3
Routing:
- net N$13: track 25.0 -> 10.0 mm
- net VBAT_OK: track 14.6 -> 10.1 mm
- net N$2: track 14.2 -> 18.5 mm
- net VBAT: track 17.5 -> 21.1 mm, vias 1 -> 2
- net VBUCK: track 69.9 -> 66.6 mm, vias 2 -> 4
- net GND: track 0.00 -> 2.86 mm, vias 0 -> 2
- net N$1: track 15.9 -> 17.9 mm
- net OUT1_M2: track 3.39 -> 5.31 mm
- net NSLEEP_M1: track 13.6 -> 11.8 mm
- net OUT3_M2: track 6.58 -> 8.40 mm
- net N$4: track 7.56 -> 5.98 mm
- net VSTOR: track 16.1 -> 14.6 mm
- net N$9: track 3.98 -> 5.47 mm
- net VHARV: track 16.8 -> 15.3 mm
- net OUT2_M2: track 5.66 -> 6.87 mm
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
Commit message: Added boardversion and fixed header spacing for wisp5
Parts:
- moved JP2 0.25 mm to (5.84, 6.86)
- moved VIN/GND 0.15 mm to (24.8, 26.7)
Other:
- board text added: "IPR board v1.0 by Koen Schaper"
Changed lines of the file:
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@@
 <setting verticaltext="up"/>
 </settings>
-<grid distance="0.01" unitdist="inch" unit="inch" style="lines" multiple="1" display="yes" altdistance="0.001" altunitdist="inch" altunit="inch"/>
+<grid distance="0.05" unitdist="inch" unit="inch" style="lines" multiple="1" display="yes" altdistance="0.005" altunitdist="inch" altunit="inch"/>
 <layers>
 <layer number="1" name="Top" color="4" fill="1" visible="yes" active="yes"/>
@@
 <layer number="20" name="Dimension" color="15" fill="1" visible="yes" active="yes"/>
 <layer number="21" name="tPlace" color="16" fill="1" visible="yes" active="yes"/>
-<layer number="22" name="bPlace" color="14" fill="1" visible="no" active="yes"/>
+<layer number="22" name="bPlace" color="14" fill="1" visible="yes" active="yes"/>
 <layer number="23" name="tOrigins" color="15" fill="1" visible="yes" active="yes"/>
 <layer number="24" name="bOrigins" color="15" fill="1" visible="yes" active="yes"/>
-<layer number="25" name="tNames" color="7" fill="1" visible="yes" active="yes"/>
+<layer number="25" name="tNames" color="7" fill="1" visible="no" active="yes"/>
 <layer number="26" name="bNames" color="7" fill="1" visible="no" active="yes"/>
 <layer number="27" name="tValues" color="7" fill="1" visible="no" active="yes"/>
@@
 <layer number="49" name="Reference" color="7" fill="1" visible="no" active="yes"/>
 <layer number="50" name="dxf" color="7" fill="1" visible="no" active="no"/>
-<layer number="51" name="tDocu" color="6" fill="1" visible="no" active="yes"/>
+<layer number="51" name="tDocu" color="6" fill="1" visible="yes" active="yes"/>
 <layer number="52" name="bDocu" color="7" fill="1" visible="no" active="yes"/>
 <layer number="53" name="tGND_GNDA" color="7" fill="9" visible="no" active="no"/>
@@
 <wire x1="30" y1="0" x2="0" y2="0" width="0.254" layer="20"/>
 <rectangle x1="5.461" y1="5.7912" x2="24.5364" y2="24.2062" layer="114"/>
+<text x="6.858" y="1.016" size="0.8128" layer="21" font="vector" ratio="12">IPR board v1.0 by Koen Schaper</text>
 </plain>
 <attributes>
@@
 <attribute name="VALUE" x="19.466" y="26.107" size="1" layer="27" ratio="11" rot="R180"/>
 </element>
-<element name="VIN/GND" library="transceiver" package="PINHEAD_1X02-1.27MM" value="PINHEAD_PINHD-1X2-1.27MM" x="24.711" y="26.854" smashed="yes" rot="R180">
-<attribute name="NAME" x="27.2002" y="29.1527" size="1" layer="25" ratio="11" rot="R180"/>
-<attribute name="VALUE" x="26.616" y="29.7115" size="1" layer="27" ratio="11" rot="R180"/>
-</element>
-<element name="JP2" library="transceiver" package="PINHEAD_1X03-1.27MM" value="PINHEAD_PINHD-1X3-1.27MM" x="6.096" y="6.858" smashed="yes" rot="R270">
-<attribute name="NAME" x="7.3533" y="8.5852" size="1" layer="25" ratio="11" rot="R270"/>
-<attribute name="VALUE" x="3.2385" y="10.033" size="1" layer="27" ratio="11" rot="R270"/>
+<element name="VIN/GND" library="transceiver" package="PINHEAD_1X02-1.27MM" value="PINHEAD_PINHD-1X2-1.27MM" x="24.7872" y="26.727" smashed="yes" rot="R180">
+<attribute name="NAME" x="27.2764" y="29.0257" size="1" layer="25" ratio="11" rot="R180"/>
+<attribute name="VALUE" x="26.6922" y="29.5845" size="1" layer="27" ratio="11" rot="R180"/>
+</element>
+<element name="JP2" library="transceiver" package="PINHEAD_1X03-1.27MM" value="PINHEAD_PINHD-1X3-1.27MM" x="5.842" y="6.858" smashed="yes" rot="R270">
+<attribute name="NAME" x="7.0993" y="8.5852" size="1" layer="25" ratio="11" rot="R270"/>
+<attribute name="VALUE" x="2.9845" y="10.033" size="1" layer="27" ratio="11" rot="R270"/>
 </element>
 <element name="JP1" library="transceiver" package="PINHEAD_1X05-1.27MM" value="PINHEAD_PINHD-1X5-1.27MM" x="9.525" y="4.572" smashed="yes">
@@
 <contactref element="U2" pad="14"/>
 <contactref element="JP2" pad="2"/>
-<wire x1="6.096" y1="8.128" x2="3.38" y2="8.128" width="0.254" layer="1"/>
+<wire x1="5.842" y1="8.128" x2="3.38" y2="8.128" width="0.254" layer="1"/>
 <wire x1="3.38" y1="8.128" x2="2.8364" y2="7.686" width="0.254" layer="1"/>
 <wire x1="5.7404" y1="1.7272" x2="26.4414" y2="1.778" width="0.254" layer="1"/>
@@
 <wire x1="24.9174" y1="6.1214" x2="23.068" y2="6.1468" width="0.254" layer="1"/>
 <wire x1="23.068" y1="6.1468" x2="23.0618" y2="6.153" width="0.254" layer="1"/>
-<wire x1="6.096" y1="8.128" x2="4.572" y2="6.604" width="0.254" layer="16"/>
+<wire x1="5.842" y1="8.128" x2="4.572" y2="6.604" width="0.254" layer="16"/>
 <wire x1="4.572" y1="6.604" x2="4.5466" y2="2.6416" width="0.254" layer="16"/>
 <via x="4.5466" y="2.6416" extent="1-16" drill="0.508"/>
@@
 <wire x1="24.9428" y1="6.8326" x2="23.1168" y2="6.8072" width="0.254" layer="1"/>
 <wire x1="23.1168" y1="6.8072" x2="23.0618" y2="6.803" width="0.254" layer="1"/>
-<wire x1="6.096" y1="6.858" x2="5.3848" y2="6.1722" width="0.254" layer="16"/>
+<wire x1="5.842" y1="6.858" x2="5.3848" y2="6.1722" width="0.254" layer="16"/>
 <wire x1="5.3848" y1="6.1722" x2="5.334" y2="2.54" width="0.254" layer="16"/>
 <wire x1="5.334" y1="2.54" x2="4.953" y2="1.397" width="0.254" layer="16"/>
@@
 <wire x1="18.191" y1="22.107" x2="19.549" y2="22.107" width="0.254" layer="1"/>
 <wire x1="19.549" y1="22.107" x2="19.558" y2="22.098" width="0.254" layer="1"/>
-<wire x1="23.441" y1="26.854" x2="23.25" y2="26.663" width="1.016" layer="1"/>
-<wire x1="23.25" y1="26.663" x2="23.25" y2="23.64355" width="1.016" layer="1"/>
+<wire x1="23.5172" y1="26.727" x2="23.5548" y2="24.4024" width="1.016" layer="1"/>
+<wire x1="23.5548" y1="24.4024" x2="23.25" y2="23.64355" width="1.016" layer="1"/>
 <wire x1="27.2914" y1="24.1308" x2="27.3304" y2="24.0918" width="0.8128" layer="1"/>
 <wire x1="27.3304" y1="24.0918" x2="27.3304" y2="21.778" width="1.016" layer="1"/>

Commit message: Changed capacitor naming, relocated part values and removed default dimension layer
Parts:
- moved C2 0.21 mm to (23.1, 9.91)
- moved R3 0.20 mm to (2.80, 2.84)
- moved R4 0.15 mm to (2.84, 6.89)
- renumbered C11 to C9, C12 to C5, C15 to C4
Routing:
- net N$1: track 17.9 -> 16.3 mm
- net VBUCK: track 66.6 -> 67.1 mm
Other:
- board size 100 x 80 mm -> 30 x 30 mm
