File: PCB/Wisp5_Harvester_Motor-driver/Wisp5_Harvester_Motor-driver.brd (EAGLE design)
At the start: 30 x 30 mm, 29 parts, among them U1 BQ25570, U2 TCA9538PWR

Commit message: Updated resistor values: VBAT_OV, VBAT_OK, VBAT_OK_HYST and VOUT
Parts:
- R1: value 8.66M -> 7.50M
- R10: value 6.49M -> 6.98M
- R2: value 4.30M -> 5.36M
- R6: value 1.82M -> 6.04M
- R7: value 5.9M -> 3.01M
- R8: value 5.49M -> 3.65M
- R9: value 6.49M -> 5.76M
Changed lines of the file:
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@@
 <setting verticaltext="up"/>
 </settings>
-<grid distance="0.01" unitdist="inch" unit="inch" style="lines" multiple="1" display="yes" altdistance="0.001" altunitdist="inch" altunit="inch"/>
+<grid distance="0.05" unitdist="inch" unit="inch" style="lines" multiple="1" display="yes" altdistance="0.005" altunitdist="inch" altunit="inch"/>
 <layers>
 <layer number="1" name="Top" color="4" fill="1" visible="yes" active="yes"/>
@@
 <attribute name="VALUE" x="5.3386" y="2.2042" size="1" layer="27" ratio="11" rot="R90"/>
 </element>
-<element name="R6" library="resistor" package="R0805" value="1.82M" x="7.336" y="26.0124" smashed="yes" rot="R270">
+<element name="R6" library="resistor" package="R0805" value="6.04M" x="7.336" y="26.0124" smashed="yes" rot="R270">
 <attribute name="NAME" x="8.3774" y="26.8252" size="1" layer="25" ratio="11" rot="R270"/>
 <attribute name="VALUE" x="4.796" y="26.6474" size="1" layer="27" ratio="11" rot="R270"/>
 </element>
-<element name="R7" library="resistor" package="R0805" value="5.9M" x="3.6864" y="26.9156" smashed="yes">
+<element name="R7" library="resistor" package="R0805" value="3.01M" x="3.6864" y="26.9156" smashed="yes">
 <attribute name="NAME" x="2.7974" y="24.8836" size="1" layer="25" ratio="11"/>
 <attribute name="VALUE" x="3.0514" y="24.3756" size="1" layer="27" ratio="11"/>
 </element>
-<element name="R8" library="resistor" package="R0805" value="5.49M" x="3.686" y="24.086" smashed="yes">
+<element name="R8" library="resistor" package="R0805" value="3.65M" x="3.686" y="24.086" smashed="yes">
 <attribute name="NAME" x="2.797" y="22.054" size="1" layer="25" ratio="11"/>
 <attribute name="VALUE" x="3.051" y="21.546" size="1" layer="27" ratio="11"/>
@@
 <attribute name="VALUE" x="0.2964" y="7.5234" size="1" layer="27" ratio="11" rot="R270"/>
 </element>
-<element name="R1" library="resistor" package="R0805" value="8.66M" x="12.1624" y="26.452" smashed="yes" rot="R180">
+<element name="R1" library="resistor" package="R0805" value="7.50M" x="12.1624" y="26.452" smashed="yes" rot="R180">
 <attribute name="NAME" x="13.0006" y="28.4586" size="1" layer="25" ratio="11" rot="R180"/>
 <attribute name="VALUE" x="12.7974" y="28.992" size="1" layer="27" ratio="11" rot="R180"/>
 </element>
-<element name="R2" library="resistor" package="R0805" value="4.30M" x="10.3004" y="22.824" smashed="yes">
+<element name="R2" library="resistor" package="R0805" value="5.36M" x="10.3004" y="22.824" smashed="yes">
 <attribute name="NAME" x="9.513" y="23.7892" size="1" layer="25" ratio="11"/>
 <attribute name="VALUE" x="9.6654" y="20.284" size="1" layer="27" ratio="11"/>
 </element>
-<element name="R10" library="resistor" package="R0805" value="6.49M" x="3.678" y="17.996" smashed="yes">
+<element name="R10" library="resistor" package="R0805" value="6.98M" x="3.678" y="17.996" smashed="yes">
 <attribute name="NAME" x="2.5096" y="15.837" size="1" layer="25" ratio="11"/>
 <attribute name="VALUE" x="3.043" y="15.456" size="1" layer="27" ratio="11"/>
 </element>
-<element name="R9" library="resistor" package="R0805" value="6.49M" x="3.651" y="21.044" smashed="yes">
+<element name="R9" library="resistor" package="R0805" value="5.76M" x="3.651" y="21.044" smashed="yes">
 <attribute name="NAME" x="2.762" y="19.012" size="1" layer="25" ratio="11"/>
 <attribute name="VALUE" x="3.016" y="18.504" size="1" layer="27" ratio="11"/>

Commit message: Increase all decoupling capacitors from 0.01uF to 0.1uF, according to the reference design of the harvester and motor driver
Parts:
- C1, C2, C4: value 0.01uF -> 0.1uF
- C7: value 0.01 uF -> 0.1 uF
Changed lines of the file:
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@@
 </autorouter>
 <elements>
-<element name="C1" library="rcl" package="C0805" value="0.01uF" x="6.801" y="14.855" smashed="yes" rot="R180">
+<element name="C1" library="rcl" package="C0805" value="0.1uF" x="6.801" y="14.855" smashed="yes" rot="R180">
 <attribute name="NAME" x="7.5376" y="13.8136" size="1" layer="25" ratio="11" rot="R180"/>
 <attribute name="VALUE" x="8.071" y="17.395" size="1" layer="27" ratio="11" rot="R180"/>
@@
 <attribute name="VALUE" x="21.3546" y="29.3234" size="1" layer="27" ratio="11" rot="R180"/>
 </element>
-<element name="C4" library="rcl" package="C0805" value="0.01uF" x="27.2914" y="25.0808" smashed="yes" rot="R90">
+<element name="C4" library="rcl" package="C0805" value="0.1uF" x="27.2914" y="25.0808" smashed="yes" rot="R90">
 <attribute name="NAME" x="29.3234" y="23.8108" size="1" layer="25" ratio="11" rot="R90"/>
 <attribute name="VALUE" x="29.8314" y="23.8108" size="1" layer="27" ratio="11" rot="R90"/>
 </element>
-<element name="C2" library="rcl" package="C0805" value="0.01uF" x="23.114" y="9.906" smashed="yes">
+<element name="C2" library="rcl" package="C0805" value="0.1uF" x="23.114" y="9.906" smashed="yes">
 <attribute name="NAME" x="22.352" y="10.922" size="1" layer="25" ratio="11"/>
 <attribute name="VALUE" x="21.844" y="7.366" size="1" layer="27" ratio="11"/>
@@
 <attribute name="VALUE" x="17.1146" y="14.8226" size="1" layer="27" ratio="11"/>
 </element>
-<element name="C7" library="rcl" package="C0805" value="0.01 uF" x="23.5472" y="17.3872" smashed="yes" rot="R180">
+<element name="C7" library="rcl" package="C0805" value="0.1 uF" x="23.5472" y="17.3872" smashed="yes" rot="R180">
 <attribute name="NAME" x="24.233" y="16.1934" size="1" layer="25" ratio="11" rot="R180"/>
 <attribute name="VALUE" x="24.8172" y="19.9272" size="1" layer="27" ratio="11" rot="R180"/>
