File: PCB/Wisp5_Harvester_Motor-driver/Wisp5_Harvester_Motor-driver.sch (EAGLE design)
At the start: 29 parts

Commit message: Redone previous work, with more focus on power routing.
Parts:
- removed R13: 1.82M, resistor:R-EU_R0805
- removed R14: 5.9M, resistor:R-EU_R0805
- removed R15: 5.49M, resistor:R-EU_R0805
- added R10: 6.49M, resistor:R-EU_R0805
- added R3, R4: 10K, resistor:R-EU_R0805
- R1: value 10K -> 8.66M
- R2: value 10K -> 4.30M
- R6: value 8.66M -> 1.82M
- R7: value 4.30M -> 5.9M
- R8: value 6.49M -> 5.49M
- renumbered U$1 to U2, U$2 to U1
Connections:
- net GND: now also R10.1, R2.1; no longer R15.1, R7.1
- net N$1: now also R10.2; no longer R8.2
- net N$10: now also R6.1, R7.2; no longer R13.1, R14.2
- net N$13: now also R1.1, R2.2; no longer R6.1, R7.2
- net N$18: now also R7.1, R8.2; no longer R14.1, R15.2
- net N$2: now also R1.2; no longer R13.2
- net SCL: now also R4.1; no longer R2.1
- net SDA: now also R3.1; no longer R1.1
- net VBUCK: now also R3.2, R4.2; no longer R1.2, R2.2
Other:
- moved on the sheet: R6, R7, R8

Commit message: Changed capacitor naming, relocated part values and removed default dimension layer
Parts:
- renumbered C11 to C9, C12 to C5, C15 to C4
Changed lines of the file:
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@@
 <grid distance="0.1" unitdist="inch" unit="inch" style="lines" multiple="1" display="no" altdistance="0.01" altunitdist="inch" altunit="inch"/>
 <layers>
-<layer number="1" name="Top" color="4" fill="1" visible="yes" active="no"/>
-<layer number="16" name="Bottom" color="1" fill="1" visible="yes" active="no"/>
-<layer number="17" name="Pads" color="2" fill="1" visible="yes" active="no"/>
-<layer number="18" name="Vias" color="2" fill="1" visible="yes" active="no"/>
-<layer number="19" name="Unrouted" color="6" fill="1" visible="yes" active="no"/>
-<layer number="20" name="Dimension" color="15" fill="1" visible="yes" active="no"/>
-<layer number="21" name="tPlace" color="16" fill="1" visible="yes" active="no"/>
-<layer number="22" name="bPlace" color="14" fill="1" visible="yes" active="no"/>
-<layer number="23" name="tOrigins" color="15" fill="1" visible="yes" active="no"/>
-<layer number="24" name="bOrigins" color="15" fill="1" visible="yes" active="no"/>
-<layer number="25" name="tNames" color="7" fill="1" visible="yes" active="no"/>
-<layer number="26" name="bNames" color="7" fill="1" visible="yes" active="no"/>
-<layer number="27" name="tValues" color="7" fill="1" visible="yes" active="no"/>
-<layer number="28" name="bValues" color="7" fill="1" visible="yes" active="no"/>
+<layer number="1" name="Top" color="4" fill="1" visible="no" active="no"/>
+<layer number="16" name="Bottom" color="1" fill="1" visible="no" active="no"/>
+<layer number="17" name="Pads" color="2" fill="1" visible="no" active="no"/>
+<layer number="18" name="Vias" color="2" fill="1" visible="no" active="no"/>
+<layer number="19" name="Unrouted" color="6" fill="1" visible="no" active="no"/>
+<layer number="20" name="Dimension" color="15" fill="1" visible="no" active="no"/>
+<layer number="21" name="tPlace" color="16" fill="1" visible="no" active="no"/>
+<layer number="22" name="bPlace" color="14" fill="1" visible="no" active="no"/>
+<layer number="23" name="tOrigins" color="15" fill="1" visible="no" active="no"/>
+<layer number="24" name="bOrigins" color="15" fill="1" visible="no" active="no"/>
+<layer number="25" name="tNames" color="7" fill="1" visible="no" active="no"/>
+<layer number="26" name="bNames" color="7" fill="1" visible="no" active="no"/>
+<layer number="27" name="tValues" color="7" fill="1" visible="no" active="no"/>
+<layer number="28" name="bValues" color="7" fill="1" visible="no" active="no"/>
 <layer number="29" name="tStop" color="7" fill="3" visible="no" active="no"/>
 <layer number="30" name="bStop" color="7" fill="6" visible="no" active="no"/>
@@
 <layer number="35" name="tGlue" color="7" fill="4" visible="no" active="no"/>
 <layer number="36" name="bGlue" color="7" fill="5" visible="no" active="no"/>
-<layer number="37" name="tTest" color="7" fill="1" visible="yes" active="no"/>
-<layer number="38" name="bTest" color="7" fill="1" visible="yes" active="no"/>
+<layer number="37" name="tTest" color="7" fill="1" visible="no" active="no"/>
+<layer number="38" name="bTest" color="7" fill="1" visible="no" active="no"/>
 <layer number="39" name="tKeepout" color="4" fill="11" visible="no" active="no"/>
 <layer number="40" name="bKeepout" color="1" fill="11" visible="no" active="no"/>
@@
 <layer number="44" name="Drills" color="7" fill="1" visible="no" active="no"/>
 <layer number="45" name="Holes" color="7" fill="1" visible="no" active="no"/>
-<layer number="46" name="Milling" color="3" fill="1" visible="yes" active="no"/>
-<layer number="47" name="Measures" color="7" fill="1" visible="yes" active="no"/>
-<layer number="48" name="Document" color="7" fill="1" visible="yes" active="no"/>
-<layer number="49" name="Reference" color="7" fill="1" visible="yes" active="no"/>
-<layer number="50" name="dxf" color="7" fill="1" visible="yes" active="no"/>
-<layer number="51" name="tDocu" color="6" fill="1" visible="yes" active="no"/>
-<layer number="52" name="bDocu" color="7" fill="1" visible="yes" active="no"/>
-<layer number="53" name="tGND_GNDA" color="7" fill="9" visible="yes" active="no"/>
-<layer number="54" name="bGND_GNDA" color="1" fill="9" visible="yes" active="no"/>
-<layer number="56" name="wert" color="7" fill="1" visible="yes" active="no"/>
-<layer number="57" name="tCAD" color="7" fill="1" visible="yes" active="no"/>
-<layer number="59" name="tCarbon" color="7" fill="1" visible="yes" active="no"/>
-<layer number="60" name="bCarbon" color="7" fill="1" visible="yes" active="no"/>
+<layer number="46" name="Milling" color="3" fill="1" visible="no" active="no"/>
+<layer number="47" name="Measures" color="7" fill="1" visible="no" active="no"/>
+<layer number="48" name="Document" color="7" fill="1" visible="no" active="no"/>
+<layer number="49" name="Reference" color="7" fill="1" visible="no" active="no"/>
+<layer number="50" name="dxf" color="7" fill="1" visible="no" active="no"/>
+<layer number="51" name="tDocu" color="6" fill="1" visible="no" active="no"/>
+<layer number="52" name="bDocu" color="7" fill="1" visible="no" active="no"/>
+<layer number="53" name="tGND_GNDA" color="7" fill="9" visible="no" active="no"/>
+<layer number="54" name="bGND_GNDA" color="1" fill="9" visible="no" active="no"/>
+<layer number="56" name="wert" color="7" fill="1" visible="no" active="no"/>
+<layer number="57" name="tCAD" color="7" fill="1" visible="no" active="no"/>
+<layer number="59" name="tCarbon" color="7" fill="1" visible="no" active="no"/>
+<layer number="60" name="bCarbon" color="7" fill="1" visible="no" active="no"/>
 <layer number="90" name="Modules" color="5" fill="1" visible="yes" active="yes"/>
 <layer number="91" name="Nets" color="2" fill="1" visible="yes" active="yes"/>
@@
 <part name="GND6" library="supply1" deviceset="GND" device=""/>
 <part name="GND7" library="supply1" deviceset="GND" device=""/>
-<part name="C12" library="rcl" deviceset="C-EU" device="C0805" value="10nF"/>
+<part name="C5" library="rcl" deviceset="C-EU" device="C0805" value="10nF"/>
 <part name="R10" library="resistor" deviceset="R-EU_" device="R0805" value="6.49M"/>
 <part name="R9" library="resistor" deviceset="R-EU_" device="R0805" value="6.49M"/>
@@
 <part name="GND12" library="supply1" deviceset="GND" device=""/>
 <part name="GND21" library="supply1" deviceset="GND" device=""/>
-<part name="C15" library="rcl" deviceset="C-EU" device="C0805" value="0.01uF"/>
-<part name="C11" library="ipr" deviceset="BZ054B223ZSBBQ" device=""/>
+<part name="C4" library="rcl" deviceset="C-EU" device="C0805" value="0.01uF"/>
+<part name="C9" library="ipr" deviceset="BZ054B223ZSBBQ" device=""/>
 <part name="GND3" library="supply1" deviceset="GND" device=""/>
 <part name="R3" library="resistor" deviceset="R-EU_" device="R0805" value="10K"/>
@@
 <instance part="GND6" gate="1" x="76.2" y="66.04"/>
 <instance part="GND7" gate="1" x="147.32" y="66.04"/>
-<instance part="C12" gate="G$1" x="63.5" y="50.8"/>
+<instance part="C5" gate="G$1" x="63.5" y="50.8"/>
 <instance part="R10" gate="G$1" x="116.84" y="10.16" rot="R90"/>
 <instance part="R9" gate="G$1" x="116.84" y="25.4" rot="R90"/>
@@
 <instance part="GND12" gate="1" x="116.84" y="38.1"/>
 <instance part="GND21" gate="1" x="76.2" y="45.72"/>
-<instance part="C15" gate="G$1" x="43.18" y="55.88"/>
-<instance part="C11" gate="G$1" x="127" y="99.06" rot="R180"/>
+<instance part="C4" gate="G$1" x="43.18" y="55.88"/>
+<instance part="C9" gate="G$1" x="127" y="99.06" rot="R180"/>
 <instance part="VIN/GND" gate="G$1" x="35.56" y="17.78"/>
 </instances>
@@
 <junction x="48.26" y="45.72"/>
 <junction x="48.26" y="45.72"/>
-<pinref part="C12" gate="G$1" pin="2"/>
+<pinref part="C5" gate="G$1" pin="2"/>
 <wire x1="48.26" y1="45.72" x2="63.5" y2="45.72" width="0.1524" layer="91"/>
 <pinref part="C3" gate="G$1" pin="2"/>
@@
 <wire x1="43.18" y1="45.72" x2="48.26" y2="45.72" width="0.1524" layer="91"/>
 <wire x1="33.02" y1="50.8" x2="33.02" y2="45.72" width="0.1524" layer="91"/>
-<pinref part="C15" gate="G$1" pin="2"/>
+<pinref part="C4" gate="G$1" pin="2"/>
 <wire x1="43.18" y1="50.8" x2="43.18" y2="45.72" width="0.1524" layer="91"/>
 <junction x="43.18" y="45.72"/>
@@
 <pinref part="U1" gate="G$1" pin="NC@17"/>
 <wire x1="116.84" y1="76.2" x2="116.84" y2="88.9" width="0.1524" layer="91"/>
-<pinref part="C11" gate="G$1" pin="GND@2"/>
+<pinref part="C9" gate="G$1" pin="GND@2"/>
 <wire x1="139.7" y1="101.6" x2="144.78" y2="101.6" width="0.127" layer="91"/>
 <wire x1="144.78" y1="101.6" x2="144.78" y2="96.52" width="0.127" layer="91"/>
-<pinref part="C11" gate="G$1" pin="GND@1"/>
+<pinref part="C9" gate="G$1" pin="GND@1"/>
 <wire x1="139.7" y1="96.52" x2="144.78" y2="96.52" width="0.127" layer="91"/>
 <wire x1="144.78" y1="96.52" x2="144.78" y2="88.9" width="0.127" layer="91"/>
@@
 <net name="N$9" class="0">
 <segment>
-<pinref part="C12" gate="G$1" pin="1"/>
+<pinref part="C5" gate="G$1" pin="1"/>
 <pinref part="U1" gate="G$1" pin="VREF_SAMP"/>
 <wire x1="63.5" y1="53.34" x2="81.28" y2="53.34" width="0.1524" layer="91"/>
@@
 <wire x1="111.76" y1="76.2" x2="111.76" y2="96.52" width="0.1524" layer="91"/>
 <label x="111.76" y="83.82" size="1.778" layer="95" rot="R90"/>
-<pinref part="C11" gate="G$1" pin="VCC"/>
+<pinref part="C9" gate="G$1" pin="VCC"/>
 <wire x1="114.3" y1="99.06" x2="111.76" y2="99.06" width="0.127" layer="91"/>
 <wire x1="111.76" y1="99.06" x2="111.76" y2="96.52" width="0.127" layer="91"/>
@@
 <wire x1="66.04" y1="76.2" x2="66.04" y2="63.5" width="0.1524" layer="91"/>
 <junction x="66.04" y="63.5"/>
-<pinref part="C15" gate="G$1" pin="1"/>
+<pinref part="C4" gate="G$1" pin="1"/>
 <wire x1="43.18" y1="58.42" x2="43.18" y2="63.5" width="0.1524" layer="91"/>
 <junction x="43.18" y="63.5"/>

Commit message: Updated resistor values: VBAT_OV, VBAT_OK, VBAT_OK_HYST and VOUT
Parts:
- R1: value 8.66M -> 7.50M
- R10: value 6.49M -> 6.98M
- R2: value 4.30M -> 5.36M
- R6: value 1.82M -> 6.04M
- R7: value 5.9M -> 3.01M
- R8: value 5.49M -> 3.65M
- R9: value 6.49M -> 5.76M
Changed lines of the file:
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@@
 <part name="GND7" library="supply1" deviceset="GND" device=""/>
 <part name="C5" library="rcl" deviceset="C-EU" device="C0805" value="10nF"/>
-<part name="R10" library="resistor" deviceset="R-EU_" device="R0805" value="6.49M"/>
-<part name="R9" library="resistor" deviceset="R-EU_" device="R0805" value="6.49M"/>
+<part name="R10" library="resistor" deviceset="R-EU_" device="R0805" value="6.98M"/>
+<part name="R9" library="resistor" deviceset="R-EU_" device="R0805" value="5.76M"/>
 <part name="GND9" library="supply1" deviceset="GND" device=""/>
 <part name="C6" library="rcl" deviceset="C-EU" device="C0805" value="4.7uF"/>
@@
 <part name="GND10" library="supply1" deviceset="GND" device=""/>
 <part name="GND11" library="supply1" deviceset="GND" device=""/>
-<part name="R2" library="resistor" deviceset="R-EU_" device="R0805" value="4.30M"/>
-<part name="R1" library="resistor" deviceset="R-EU_" device="R0805" value="8.66M"/>
+<part name="R2" library="resistor" deviceset="R-EU_" device="R0805" value="5.36M"/>
+<part name="R1" library="resistor" deviceset="R-EU_" device="R0805" value="7.50M"/>
 <part name="L1" library="passives" deviceset="COILCRAFT-LPS4018" device="" value="22uH"/>
 <part name="L2" library="passives" deviceset="COILCRAFT-LPS4018" device="" value="10uH"/>
 <part name="C8" library="rcl" deviceset="C-EU" device="C0805" value="22uF"/>
-<part name="R6" library="resistor" deviceset="R-EU_" device="R0805" value="1.82M"/>
-<part name="R7" library="resistor" deviceset="R-EU_" device="R0805" value="5.9M"/>
-<part name="R8" library="resistor" deviceset="R-EU_" device="R0805" value="5.49M"/>
+<part name="R6" library="resistor" deviceset="R-EU_" device="R0805" value="6.04M"/>
+<part name="R7" library="resistor" deviceset="R-EU_" device="R0805" value="3.01M"/>
+<part name="R8" library="resistor" deviceset="R-EU_" device="R0805" value="3.65M"/>
 <part name="GND12" library="supply1" deviceset="GND" device=""/>
 <part name="GND21" library="supply1" deviceset="GND" device=""/>

Commit message: Increase all decoupling capacitors from 0.01uF to 0.1uF, according to the reference design of the harvester and motor driver
Parts:
- C1, C2, C4: value 0.01uF -> 0.1uF
- C7: value 0.01 uF -> 0.1 uF
Changed lines of the file:
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@@
 <part name="GND9" library="supply1" deviceset="GND" device=""/>
 <part name="C6" library="rcl" deviceset="C-EU" device="C0805" value="4.7uF"/>
-<part name="C7" library="rcl" deviceset="C-EU" device="C0805" value="0.01 uF"/>
+<part name="C7" library="rcl" deviceset="C-EU" device="C0805" value="0.1 uF"/>
 <part name="GND10" library="supply1" deviceset="GND" device=""/>
 <part name="GND11" library="supply1" deviceset="GND" device=""/>
@@
 <part name="GND12" library="supply1" deviceset="GND" device=""/>
 <part name="GND21" library="supply1" deviceset="GND" device=""/>
-<part name="C4" library="rcl" deviceset="C-EU" device="C0805" value="0.01uF"/>
+<part name="C4" library="rcl" deviceset="C-EU" device="C0805" value="0.1uF"/>
 <part name="C9" library="ipr" deviceset="BZ054B223ZSBBQ" device=""/>
 <part name="GND3" library="supply1" deviceset="GND" device=""/>
@@
 <part name="GND4" library="supply1" deviceset="GND" device=""/>
 <part name="GND13" library="supply1" deviceset="GND" device=""/>
-<part name="C2" library="rcl" deviceset="C-EU" device="C0805" value="0.01uF"/>
-<part name="C1" library="rcl" deviceset="C-EU" device="C0805" value="0.01uF"/>
+<part name="C2" library="rcl" deviceset="C-EU" device="C0805" value="0.1uF"/>
+<part name="C1" library="rcl" deviceset="C-EU" device="C0805" value="0.1uF"/>
 <part name="VIN/GND" library="transceiver" deviceset="PINHEAD_PINHD-1X2-1.27MM" device=""/>
 <part name="U2" library="ipr" deviceset="TCA9538PWR" device=""/>
