File: PCB/Wisp5_Harvester_Motor-driver_V2/Wisp5_Harvester_Motor-driver_V2.brd (EAGLE design)
At the start: 30 x 30 mm, 30 parts, among them M1 PINHEAD_PINHD-1X2-1.27MM, M2 PINHEAD_PINHD-1X2-1.27MM, U1 BQ25570, U2 BGM250, U3 DRV8836

Commit message: Fix battery header orientation!
Parts:
- moved VBAT/GND 1.31 mm to (27.5, 3.30), turned to 180 degrees
Routing:
- net VBOOST: track 12.7 -> 9.92 mm
Changed lines of the file:
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@@
 <attribute name="VALUE" x="16.984" y="24.0682" size="0.8" layer="27" rot="R180"/>
 </element>
-<element name="VBAT/GND" library="Wisp5_Harvester_Motor-driver_V2" package="PINHEAD_1X02-1.27MM" value="PINHEAD_PINHD-1X2-1.27MM" x="26.14" y="3.306" smashed="yes">
-<attribute name="NAME" x="23.3588" y="4.6173" size="0.8" layer="25" ratio="10"/>
+<element name="VBAT/GND" library="Wisp5_Harvester_Motor-driver_V2" package="PINHEAD_1X02-1.27MM" value="PINHEAD_PINHD-1X2-1.27MM" x="27.454" y="3.298" smashed="yes" rot="R180">
+<attribute name="NAME" x="29.3462" y="5.4411" size="0.8" layer="25" ratio="10" rot="R180"/>
 </element>
 <element name="VIN/GND" library="Wisp5_Harvester_Motor-driver_V2" package="PINHEAD_1X02-1.27MM" value="PINHEAD_PINHD-1X2-1.27MM" x="26.138" y="26.992" smashed="yes" rot="R180">
@@
 <contactref element="WISP" pad="VBOOST"/>
 <contactref element="VBAT/GND" pad="2"/>
-<wire x1="16.7767" y1="3.302" x2="23.368" y2="3.302" width="0.4064" layer="1"/>
-<wire x1="23.368" y1="3.302" x2="25.146" y2="5.08" width="0.4064" layer="1"/>
-<wire x1="25.146" y1="5.08" x2="26.67" y2="5.08" width="0.4064" layer="1"/>
-<wire x1="26.67" y1="5.08" x2="27.432" y2="4.318" width="0.4064" layer="1"/>
-<wire x1="27.432" y1="4.318" x2="27.432" y2="3.328" width="0.4064" layer="1"/>
-<wire x1="27.432" y1="3.328" x2="27.41" y2="3.306" width="0.254" layer="1"/>
+<wire x1="16.7767" y1="3.302" x2="22.86" y2="3.302" width="0.4064" layer="1"/>
+<wire x1="22.86" y1="3.302" x2="23.368" y2="3.302" width="0.4064" layer="1"/>
+<wire x1="22.86" y1="3.302" x2="26.18" y2="3.302" width="0.4064" layer="1"/>
+<wire x1="26.18" y1="3.302" x2="26.184" y2="3.298" width="0.4064" layer="1"/>
 </signal>
 <signal name="SCL">
